File: PCB/bass.kicad_sch (KiCad schematic)
At the start: 66 parts, among them U1Unit OPA2134PA, U2Unit NJM4556AD, U3 TLE2426CLP

Commit message: progress!
Parts:
- C3: symbol Device:C -> Device:C_Polarized
Connections:
- net +9V: now reaches C2.1
- net +9V: now also C1.1, C_byp_U1.1, C_byp_U2.1, C_pwr_U1.1, C_pwr_U2.1, J_SWITCH.4 (Pin_4), R_LED.1, R_damp.2, TP1.1, U1Unit.8 (V+), U2Unit.8 (V+)
- net GND: now reaches C2.2
- net GND: now also C1.2, C3.2, C4.2, C_bias.2, C_byp_U1.2, C_byp_U2.2, C_pwr_U1.2, C_pwr_U2.2, C_vref_U1.2, C_vref_U2.2, H1.1, H2.1, H3.1, H4.1, J_LED.2 (Pin_2), J_LINE_OUT.2 (Pin_2), J_PICKUP.2 (Pin_2), J_VOL_POT.1 (Pin_1), PWR_IN.2 (Pin_2), R_bleed1.2, R_bleed2.2, TP2.1, U1Unit.4 (V-), U2Unit.4 (V-)
- net at U1Unit.1: now also R2.1, U1Unit.2 (-)
- net at U1Unit.3 (+): now also C_in.2, R1.1
- net at R_damp.1: now also L1.2
- net NODE_B: now reaches R_treble2.1
- net NODE_B: now also C_vol.1, R_bass2.1, R_flat_fb.2, TP5.1, U1Unit.7
- net at R_treble2.2: now also J_TREB_POT.1 (Pin_1)
- net at J_HP_OUT.1 (Pin_1): now also C_hp_out1.2, R_bleed1.1
- net at J_HP_OUT.2 (Pin_2): now also C_hp_out2.2, R_bleed2.1
- net at R_treble3.1: now also J_BASS_POT.2 (Pin_2), R_flat_fb.1, R_flat_in.1, U1Unit.6 (-)
- net at R_treble3.2: now also C_treble.2
- net VREF: now reaches R1.2
- net VREF: now also C3.1, C4.1, C_vref_U1.1, C_vref_U2.1, R1.2, R_bias.2, R_bias_hp1.2, R_bias_hp2.2, R_gain1.2, R_gain2.2, TP3.1
- net at PWR_IN.1 (Pin_1): now also D1.2 (A)
- net at J_TREB_POT.2 (Pin_2): now also C_treble.1
- net at J_TREB_POT.3 (Pin_3): now also R_treble1.2
- net at J_PICKUP.1 (Pin_1): now also R_in_prot.1
- net at J_BASS_POT.1 (Pin_1): now also R_bass2.2
- net at J_BASS_POT.3 (Pin_3): now also R_bass1.2
- net at R_LED.2: now also J_LED.1 (Pin_1)
- net NODE_C: now reaches C_hp_in1.1
- net NODE_C: now also C_hp_in2.1, J_LINE_OUT.1 (Pin_1), J_VOL_POT.2 (Pin_2), TP6.1
- net at C_hp_in1.2: now also R_bias_hp1.1, U2Unit.3 (+)
- net at U1Unit.5 (+): now also C_bias.1, R_bias.1
- net at C_hp_out1.1: now also R8.2
- net at R_fb1.1: now also R_gain1.1, U2Unit.2 (-)
- net at R_fb1.2: now also R8.1, U2Unit.1
- net NODE_A: now reaches R_flat_in.2
- net NODE_A: now also R2.2, R_bass1.1, R_treble1.1, TP4.1
- net at R_bias_hp2.1: now also C_hp_in2.2, U2Unit.5 (+)
- net at D1.1 (K): now also L1.1
- net at R_gain2.1: now also R_fb2.1, U2Unit.6 (-)
- net at C_vol.2: now also J_SWITCH.1 (Pin_1)
- net at J_VOL_POT.3 (Pin_3): now also J_SWITCH.2 (Pin_2)
- net at R_in_prot.2: now also C_in.1
- net at R_fb2.2: now also R11.1, U2Unit.7
- net at C_hp_out2.1: now also R11.2
- net PICKUP_HOT: now reaches J_SWITCH.3 (Pin_3)
- no-connect marks 0 -> 2
Other:
- moved on the sheet: C_bias, C_byp_U2, C_hp_in2, C_hp_out1, C_hp_out2, C_pwr_U2, C_treble, C_vref_U2, H1, H2, H3, H4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

Commit message: progresse
Parts:
- C1, C_pwr_U1, C_pwr_U2: footprint (none) -> Capacitor_THT:CP_Radial_D8.0mm_P3.50mm
- C2, C4, C_byp_U1, C_byp_U2, C_vref_U1, C_vref_U2: footprint (none) -> Capacitor_THT:C_Disc_D5.0mm_W2.5mm_P5.00mm
- C3: footprint (none) -> Capacitor_THT:CP_Radial_D12.5mm_P5.00mm
- C_bias1: renamed from C_bias; footprint (none) -> Capacitor_THT:C_Disc_D5.0mm_W2.5mm_P5.00mm
- C_hp_in1, C_hp_in2: footprint (none) -> Capacitor_THT:C_Rect_L7.2mm_W2.5mm_P5.00mm_FKS2_FKP2_MKS2_MKP2
- C_hp_out1, C_hp_out2: footprint (none) -> Capacitor_THT:CP_Radial_D10.0mm_P5.00mm
- C_in1: renamed from C_in; footprint (none) -> Capacitor_THT:C_Rect_L7.2mm_W2.5mm_P5.00mm_FKS2_FKP2_MKS2_MKP2
- C_treble1: renamed from C_treble; footprint (none) -> Capacitor_THT:C_Rect_L7.2mm_W2.5mm_P5.00mm_FKS2_FKP2_MKS2_MKP2
- C_vol1: renamed from C_vol; footprint (none) -> Capacitor_THT:C_Rect_L13.5mm_W5.0mm_P10.00mm_FKS3_FKP3_MKS4
- D1: footprint (none) -> Diode_THT:D_DO-41_SOD81_P10.16mm_Horizontal
- H1, H2, H3, H4: footprint (none) -> MountingHole:MountingHole_3.2mm_M3_Pad
- J_BASS_POT1: renamed from J_BASS_POT; footprint (none) -> Connector_PinHeader_2.54mm:PinHeader_1x03_P2.54mm_Vertical
- J_HP_OUT1: renamed from J_HP_OUT; footprint (none) -> Connector_PinHeader_2.54mm:PinHeader_1x03_P2.54mm_Vertical
- J_LED1: renamed from J_LED; footprint (none) -> Connector_PinHeader_2.54mm:PinHeader_1x02_P2.54mm_Vertical
- J_LINE_OUT1: renamed from J_LINE_OUT; footprint (none) -> Connector_PinHeader_2.54mm:PinHeader_1x02_P2.54mm_Vertical
- J_PICKUP1: renamed from J_PICKUP; footprint (none) -> Connector_PinHeader_2.54mm:PinHeader_1x02_P2.54mm_Vertical
- J_SWITCH1: renamed from J_SWITCH; footprint (none) -> Connector_PinHeader_2.54mm:PinHeader_1x06_P2.54mm_Vertical
- J_TREB_POT1: renamed from J_TREB_POT; footprint (none) -> Connector_PinHeader_2.54mm:PinHeader_1x03_P2.54mm_Vertical
- J_VOL_POT1: renamed from J_VOL_POT; footprint (none) -> Connector_PinHeader_2.54mm:PinHeader_1x03_P2.54mm_Vertical
- L1: footprint (none) -> Inductor_THT:L_Radial_D10.0mm_P5.00mm_Fastron_07M
- PWR_IN1: renamed from PWR_IN; footprint (none) -> Connector_PinHeader_2.54mm:PinHeader_1x02_P2.54mm_Vertical
- R1, R11, R2, R8, R_bass1, R_bass2, R_bias_hp1, R_bias_hp2, R_bleed1, R_bleed2, R_fb1, R_fb2, R_gain1, R_gain2, R_treble1, R_treble2, R_treble3: footprint (none) -> Resistor_THT:R_Axial_DIN0207_L6.3mm_D2.5mm_P10.16mm_Horizontal
- R_LED1: renamed from R_LED; footprint (none) -> Resistor_THT:R_Axial_DIN0207_L6.3mm_D2.5mm_P10.16mm_Horizontal
- R_bias1: renamed from R_bias; footprint (none) -> Resistor_THT:R_Axial_DIN0207_L6.3mm_D2.5mm_P10.16mm_Horizontal
- R_damp1: renamed from R_damp; footprint (none) -> Resistor_THT:R_Axial_DIN0207_L6.3mm_D2.5mm_P10.16mm_Horizontal
- R_flat_fb1: renamed from R_flat_fb; footprint (none) -> Resistor_THT:R_Axial_DIN0207_L6.3mm_D2.5mm_P10.16mm_Horizontal
- R_flat_in1: renamed from R_flat_in; footprint (none) -> Resistor_THT:R_Axial_DIN0207_L6.3mm_D2.5mm_P10.16mm_Horizontal
- R_in_prot1: renamed from R_in_prot; footprint (none) -> Resistor_THT:R_Axial_DIN0207_L6.3mm_D2.5mm_P10.16mm_Horizontal
- R_stab1: renamed from R1; footprint (none) -> Resistor_THT:R_Axial_DIN0207_L6.3mm_D2.5mm_P10.16mm_Horizontal
- TP1, TP2, TP3, TP4, TP5, TP6: footprint (none) -> TestPoint:TestPoint_Pad_2.0x2.0mm
- U1: renamed from U1Unit; footprint (none) -> Package_DIP:DIP-8_W7.62mm
- U1: renamed from U1Unit; value OPA2134 -> OPA2134PA; footprint (none) -> Package_DIP:DIP-8_W7.62mm
- U2Unit1: renamed from U2Unit; footprint (none) -> Package_DIP:DIP-8_W7.62mm
- U3: footprint (none) -> Package_TO_SOT_THT:TO-92_Inline
Connections:
- net +9V: now also U3.3 (IN)
- net GND: now also J_HP_OUT1.3 (Pin_3), U3.2 (GND)
- net PICKUP_HOT: now also J_PICKUP1.1 (Pin_1), R_in_prot1.1
- net at R_stab1.1: now also U3.1 (OUT)

Commit message: .
Parts:
- renumbered U2Unit1 to U2
Changed lines of the file:
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@@
 		(dnp no)
 		(fields_autoplaced yes)
-		(property "Reference" "U2Unit1"
+		(property "Reference" "U2"
 			(at 246.38 95.2499 0)
 			(effects
@@
 			(project ""
 				(path "/9a75853d-3653-4ddd-a04a-f8cd049113a5"
-					(reference "U2Unit1")
+					(reference "U2")
 					(unit 3)
 				)
@@
 		(dnp no)
 		(fields_autoplaced yes)
-		(property "Reference" "U2Unit1"
+		(property "Reference" "U2"
 			(at 265.43 16.51 0)
 			(effects
@@
 			(project ""
 				(path "/9a75853d-3653-4ddd-a04a-f8cd049113a5"
-					(reference "U2Unit1")
+					(reference "U2")
 					(unit 2)
 				)
@@
 		(dnp no)
 		(fields_autoplaced yes)
-		(property "Reference" "U2Unit1"
+		(property "Reference" "U2"
 			(at 219.71 20.32 0)
 			(effects
@@
 			(project ""
 				(path "/9a75853d-3653-4ddd-a04a-f8cd049113a5"
-					(reference "U2Unit1")
+					(reference "U2")
 					(unit 1)
 				)
